Commit message: feat:完善了urdf文件和rviz2的配置
1. 通过SolidWorks的插件,现在urdf文件内包含了更多的link与joint以及对应的参数
2. rviz2新建了更好的默认显示配置

File: ros2_jazzy/src/yuangod_description/urdf/urdf/yuangod_smart_car.urdf (robot description, URDF)
Before this commit: robot yuangod_smart_car, 3 links, 2 joints
Links:
- removed link base_footprint
- removed link lidar_link
- added link camera_Link, mass 0.00265119308085073; collision mesh filename=package://yuangod_description/meshes/camera_Link.STL; visual mesh filename=package://yuangod_description/meshes/camera_Link.STL
- added link laser_Link, mass 0.0254427990392578; collision mesh filename=package://yuangod_description/meshes/laser_Link.STL; visual mesh filename=package://yuangod_description/meshes/laser_Link.STL
- added link pcb_link, mass 0.00718806747239929; collision mesh filename=package://yuangod_description/meshes/pcb_link.STL; visual mesh filename=package://yuangod_description/meshes/pcb_link.STL
- added link wheel_left_link, mass 0.020267; collision mesh filename=package://yuangod_description/meshes/wheel_left_link.STL; visual mesh filename=package://yuangod_description/meshes/wheel_left_link.STL
- added link wheel_right_link, mass 0.020267; collision mesh filename=package://yuangod_description/meshes/wheel_right_link.STL; visual mesh filename=package://yuangod_description/meshes/wheel_right_link.STL
- link base_link: mass 0.180022847554128 -> 0.104620329652192
Joints:
- removed joint baselink2basefootprint
- removed joint lidar_link2base_link
- added joint camera_joint: type fixed, parent base_link, child camera_Link, origin xyz=0.05872 1.2794E-05 0.04045 rpy=0 0 0, axis 0 0 0
- added joint laser_joint: type fixed, parent base_link, child laser_Link, origin xyz=0.0091199 0 0.050659 rpy=0 0 0, axis 0 0 0
- added joint pcb_joint: type fixed, parent base_link, child pcb_link, origin xyz=-0.025278 4.1266E-05 0.019586 rpy=0 0 0, axis 0 0 0
- added joint wheel_left_joint: type continuous, parent base_link, child wheel_left_link, origin xyz=0.015133 0.035405 0.018 rpy=0 0 0, axis 0 1 0
- added joint wheel_right_joint: type continuous, parent base_link, child wheel_right_link, origin xyz=0.014933 -0.034698 0.018 rpy=0 0 0, axis 0 1 0
